Commit message: feat(urdf): mount arms flush+low on lift carriage; arms-up home pose
Remove the OpenArm "body" extrusion (openarm_body_link0) and bolt both arm
bases directly onto the moving lift carriage (lift_link), then lower them a
further 2 in (0.0508 m) per request. Arm bases now sit ~0.749 m lower than the
original extrusion mount (world z 0.629 at lift=0); the 0.85 m lift travel more
than covers the drop, inter-arm spacing unchanged (62 mm). Purely a structural
FK change (verified exact to ~1e-18, no orientation leak).

Add an arms-up HOME startup pose (HOME_CONFIG in isaac/ros_sim.py, set as the
initial joint state + drive targets; mirrored in the MoveIt SRDF "home"
group_states): all-zeros folds the now-low arms into the drivebase, so the sim
seeds an arms-up ready pose clear of the base (>0.4 m from the base box,
self-clearance >24 mm).

Ripple fixes: SRDF disable_collisions re-pointed from the removed body to
lift_link; web-viz manifest.json drops the dead body_link0 mesh entry.

Refresh geometry-dependent TEST FIXTURES for the lower workspace (fixtures, not
solver changes): _solver_test far-jump held-arm gate -> settled<2mm +
transient<80mm; _solver_test_positions grid accuracy gate robust to ~1
near-boundary point; trajectory single+dual smoke goals re-aimed to open space
(the lower mount made the old downward/inward goals unavoidable task-coupled
collisions). All 10 gated suites green.

Isaac USD (assets/usd/, gitignored) regenerated from the URDF via
isaac/convert_urdf_to_usd.py; ros_sim.py builds the ROS-bridge graph at runtime
so re-converting loses nothing.

Co-Authored-By: Claude Opus 4.8 (1M context) <noreply@anthropic.com>

File: assets/ranger_air_description/urdf/ranger_air_description.urdf (robot description, URDF)
Before this commit: robot ranger_air_description, 36 links, 35 joints
Links:
- removed link openarm_body_link0
Joints:
- removed joint openarm_mount_joint
- joint openarm_left_base_link_mount_joint: origin xyz=0.0 0.031 0.698 rpy=0.0 0.0 0.0 -> xyz=0.0135 0.19 0.3492 rpy=0.0 0.0 -1.5707963267949; parent openarm_body_link0 -> lift_link
- joint openarm_right_base_link_mount_joint: origin xyz=0.0 -0.031 0.698 rpy=0.0 0.0 0.0 -> xyz=-0.0485 0.19 0.3492 rpy=0.0 0.0 -1.5707963267949; parent openarm_body_link0 -> lift_link

Commit message: fix(sim): realistic 63kg base mass so the robot stops tipping over
Operator report: "the solver fails to converge on some positions" -- the arm sat
~80-135mm short of high/forward targets. Root cause was NOT the solver, collision,
or gravity; the whole robot was TIPPING OVER in the sim.

Investigation (tools left at repo root):
- solver reaches those exact targets to 0.0mm offline (even from the live config);
- self_collision is OFF in the Isaac import, and a Drake real-mesh probe found only
  constant mount overlaps (no config-dependent self-collision);
- Drake gravity torque is ~7 N·m vs the 40 N·m joint limit (not gravity-infeasible);
- joint1 effort pinned at its -40 N·m limit, arm dead-steady 134mm short -> a
  contact reaction; the Isaac GUI showed the robot had fallen over, arm on the floor.

base_link mass was a 9.63 kg PLACEHOLDER, leaving the free-standing base top-heavy
(lift+arms ~15kg up to ~1m over a 0.39x0.34m wheel footprint); a high/forward dual
reach pushed the combined COM past the support edge and toppled it. So certain
targets "failed" = the COM-shifting reaches that tip it.

Fix: set base_link to a realistic 63 kg (real AgileX Ranger Air) + a ~0.5x0.4x0.25m
box inertia, COM kept low (z~0.14). Mass-only is a dynamics change, so the kinematic
ROS stack + all gated suites are unaffected. Isaac loads the USD (gitignored, local),
so re-run `isaac/convert_urdf_to_usd.py` after this. Verified upright: the same
previously-failing target now reaches 7.6mm / 13.7mm with joint1 at its ~7 N·m
gravity load (was 134/80mm, saturated). (Also fixed a `--` inside the new XML comment
that Isaac tolerated but the ROS XML parser rejected.)

Diagnostic tooling added: _solver_failure_logger.py (live reach-error + joint-effort
logger), _reproduce_failures.py, _probe_cmd_vs_meas.py, _diag_contact.py,
_gravity_torque.py, _gravity_drake.py, _drake_mesh_collision_probe.py, and
tools/convert_collision_meshes.py (.dae/.stl -> Drake-loadable .obj, for if
collision-aware control is pursued later).

Co-Authored-By: Claude Opus 4.8 (1M context) <noreply@anthropic.com>

File: assets/ranger_air_description/urdf/ranger_air_description.urdf (robot description, URDF)
Before this commit: robot ranger_air_description, 35 links, 34 joints
Links:
- link base_link: mass 9.62557497725158 -> 63.0
